Commit message: ur_camera gazebo

File: src/realsense-ros/realsense2_description/urdf/_d435.urdf.xacro (robot description, xacro)
@@ -42,8 +42,8 @@
     <link name="${name}_link">
       <visual>
-        <origin xyz="${d435_cam_mount_from_center_offset} ${-d435_cam_depth_py} 0" rpy="${M_PI/2} 0 ${M_PI/2}"/>
+        <origin xyz="${d435_cam_mount_from_center_offset} ${-d435_cam_depth_py} 0" rpy="${M_PI} 0 ${M_PI/2}"/>
         <geometry>
           <!-- <box size="${d435_cam_width} ${d435_cam_height} ${d435_cam_depth}"/> -->
-	        <mesh filename="package://realsense2_description/meshes/d435.dae" />
+	        <mesh filename="package://realsense2_description/meshes/d435.obj" />
         </geometry>
       </visual>

File: src/ur_camera/urdf/realsense.gazebo.urdf.xacro (robot description, xacro)
@@ -1,8 +1,8 @@
 <?xml version="1.0"?>
 <robot xmlns:xacro="http://ros.rog/wiki/xacro">
-    <gazebo reference="connect_link">
-        <material>Gazebo/Black</material>
+    <gazebo reference="camera_link">
+        <material>Gazebo/Grey</material>
     </gazebo>
-    <xacro:macro name="realsense_ir_gazebo" params="link_name frame_name camera_name">
+    <xacro:macro name="realsense_gazebo" params="link_name frame_name camera_name">
         <gazebo reference="${link_name}">
             <sensor type="depth" name="realsense_ir_sensor">
@@ -12,5 +12,5 @@
                     <horizontal_fov>1.047</horizontal_fov>
                     <image>
-                        <format>L8</format>
+                        <format>B8G8R8</format>
                         <width>640</width>
                         <height>480</height>
@@ -21,5 +21,28 @@
                     </clip>
                 </camera>
-                <plugin name="${link_name}_controller"
+                <plugin name="${link_name}_controller" filename="libgazebo_ros_openni_kinect.so">
+                    <baseline>0.2</baseline>
+                    <alwaysOn>true</alwaysOn>
+                    <updateRate>1.0</updateRate>
+                    <cameraName>${camera_name}</cameraName>
+                    <imageTopicName>/${camera_name}/color/image_raw</imageTopicName>
+                    <cameraInfoTopicName>/${camera_name}/color/camera_info</cameraInfoTopicName>
+                    <depthImageTopicName>/${camera_name}/depth/image_raw</depthImageTopicName>
+                    <depthImageInfoTopicName>/${camera_name}/depth/camera_info</depthImageInfoTopicName>
+                    <pointCloudTopicName>/${camera_name}/depth/points</pointCloudTopicName>
+                    <frameName>${frame_name}</frameName>
+                    <pointCloudCutoff>0.5</pointCloudCutoff>
+                    <pointCloudCutoffMax>3.0</pointCloudCutoffMax>
+                    <distortionK1>0.00000001</distortionK1>
+                    <distortionK2>0.00000001</distortionK2>
+                    <distortionK3>0.00000001</distortionK3>
+                    <distortionT1>0.00000001</distortionT1>
+                    <distortionT2>0.00000001</distortionT2>
+                    <CxPrime>0</CxPrime>
+                    <Cx>0</Cx>
+                    <Cy>0</Cy>
+                    <focalLength>0</focalLength>
+                    <hackBaseline>0</hackBaseline>
+                </plugin>
             </sensor>
         </gazebo>

File: src/ur_camera/urdf/ur_with_camera.urdf.xacro (robot description, xacro)
@@ -6,4 +6,5 @@
   <xacro:include filename="$(find ur_e_description)/urdf/ur5e.urdf.xacro" />
   <xacro:include filename="$(find realsense2_description)/urdf/_d435.urdf.xacro" />
+  <xacro:include filename="$(find ur_camera)/urdf/realsense.gazebo.urdf.xacro"/>
   <xacro:property name="M_PI" value="3.1415926535897931" />
   <!-- arm -->
@@ -27,3 +28,4 @@
     <origin xyz="0.0 0.0 0.0" rpy="0.0 0.0 0.0" />
   </joint>
+  <xacro:realsense_gazebo link_name="camera_depth_frame" frame_name="realsense_optical_frame" camera_name="camera" />
 </robot>
