Commit message: add gazebo simulation

File: src/ur5e_open_door_demo/urdf/chassis.gazebo.xacro (robot description, xacro)
@@ -3,13 +3,13 @@
   <xacro:macro name="chassis_gazebo" params="prefix_chassis">
     <gazebo reference="${prefix_chassis}bottom_pan">
-      <selfCollide>true</selfCollide>
+      <!-- <selfCollide>true</selfCollide> -->
       <material>Gazebo/Black</material>
     </gazebo>
     <gazebo reference="${prefix_chassis}connect_pan">
-      <selfCollide>true</selfCollide>
+      <!-- <selfCollide>true</selfCollide> -->
       <material>Gazebo/Black</material>
     </gazebo>
     <gazebo reference="${prefix_chassis}up_pan">
-      <selfCollide>true</selfCollide>
+      <!-- <selfCollide>true</selfCollide> -->
       <material>Gazebo/Black</material>
     </gazebo>

File: src/ur5e_open_door_demo/urdf/chassis.urdf.xacro (robot description, xacro)
@@ -32,8 +32,9 @@
         <!-- link robot for ur5e with chassis -->
         <link name="${prefix}robot" />
-        <link name="${prefix}world" />
+        <!-- using in Gazebo to Fixed-->
+        <link name="world" />
         <joint name="world_bottom_joint" type="fixed">
             <origin xyz="0 0 0.009" rpy="0 0 0" />
-            <parent link="${prefix}world" />
+            <parent link="world" />
             <child link="${prefix}bottom_pan" />
         </joint>
@@ -53,4 +54,5 @@
             <child link="${prefix}robot" />
         </joint>
+        <xacro:chassis_gazebo prefix_chassis="${prefix}" />
     </xacro:macro>
 </robot>
