Commit message: add hand and gazebo_ros_ft_sensor

File: src/fmauch_universal_robot/ur_e_description/urdf/common.gazebo.xacro (robot description, xacro)
@@ -1,4 +1,7 @@
 <?xml version="1.0"?>
 <robot xmlns:xacro="http://ros.org/wiki/xacro">
+  <gazebo reference="wrist_3_link-tool0_fixed_joint">
+    <provideFeedback>true</provideFeedback>
+  </gazebo>
   <gazebo>
     <plugin name="ros_control" filename="libgazebo_ros_control.so">
@@ -6,5 +9,10 @@
       <!--robotSimType>gazebo_ros_control/DefaultRobotHWSim</robotSimType-->
     </plugin>
-<!--
+    <!-- <plugin name="ft_sensor" filename="libgazebo_ros_ft_sensor.so">
+      <updateRate>100.0</updateRate>
+      <topicName>/wrench</topicName>
+      <jointName>wrist_3_link-tool0_fixed_joint</jointName>
+    </plugin> -->
+    <!--
     <plugin name="gazebo_ros_power_monitor_controller" filename="libgazebo_ros_power_monitor.so">
       <alwaysOn>true</alwaysOn>
