Commit message: add hand and gazebo_ros_ft_sensor

File: src/ur5e_open_door_demo/urdf/ur5e_with_chassis.urdf.xacro (robot description, xacro)
@@ -18,3 +18,42 @@
         <child link="${prefix_robot}base_link" />
     </joint>
+    <link name="${prefix_robot}hand_link">
+        <visual>
+            <origin xyz="0 0 0" rpy="0 0 0" />
+            <geometry>
+                <mesh filename="package://ur5e_open_door_demo/meshes/hand.STL" scale="1 1 1" />
+            </geometry>
+            <material name="LightGrey">
+                <color rgba="0.7 0.7 0.7 1.0" />
+            </material>
+        </visual>
+        <collision>
+            <origin xyz="0 0 0" rpy="0 0 0" />
+            <geometry>
+                <mesh filename="package://ur5e_open_door_demo/meshes/hand.STL" scale="1 1 1" />
+            </geometry>
+        </collision>
+        <xacro:cylinder_inertial radius="0.045" length="0.05" mass="0.1">
+            <origin xyz="0.0 0.0 ${-0.05/2}" rpy="0 0 0" />
+        </xacro:cylinder_inertial>
+    </link>
+    <joint name="tool0_hand_joint" type="fixed">
+        <limit velocity="6.5" effort="1000" />
+        <origin xyz="0 0 0" rpy="0 0 0" />
+        <parent link="${prefix_robot}tool0" />
+        <child link="${prefix_robot}hand_link" />
+    </joint>
+    <gazebo reference="${prefix_robot}wrist_3_joint">
+        <provideFeedback>true</provideFeedback>
+    </gazebo>
+    <gazebo reference="${prefix_robot}hand_link">
+        <material>Gazebo/Grey</material>
+    </gazebo>
+    <gazebo>
+        <plugin name="ft_sensor" filename="libgazebo_ros_ft_sensor.so">
+            <updateRate>100.0</updateRate>
+            <topicName>wrench</topicName>
+            <jointName>${prefix_robot}wrist_3_joint</jointName>
+        </plugin>
+    </gazebo>
 </robot>
